Commit message: 更新arm的有机械限位的urdf和mjcf+obj

File: src/runtime/sim/model/rm26_engineer_description/rm26_arm.urdf (robot description, URDF)
Before this commit: robot GC, 12 links, 11 joints
Links:
- link base_link: geometry collision mesh filename=package://GC3.1/meshes/base_link.STL; visual mesh filename=package://GC3.1/meshes/base_link.STL
- link line_link: geometry collision mesh filename=package://GC3.1/meshes/line_link.STL; visual mesh filename=package://GC3.1/meshes/line_link.STL
- link link_1: geometry collision mesh filename=package://GC3.1/meshes/link_1.STL; visual mesh filename=package://GC3.1/meshes/link_1.STL
- link link_2: mass 0.58398682899762 -> 0.583986828997619; geometry collision mesh filename=package://GC3.1/meshes/link_2.STL; visual mesh filename=package://GC3.1/meshes/link_2.STL
- link link_3: geometry collision mesh filename=package://GC3.1/meshes/link_3.STL; visual mesh filename=package://GC3.1/meshes/link_3.STL
- link link_4: mass 0.263988174644702 -> 0.263988174644703; geometry collision mesh filename=package://GC3.1/meshes/link_4.STL; visual mesh filename=package://GC3.1/meshes/link_4.STL
- link link_5: geometry collision mesh filename=package://GC3.1/meshes/link_5.STL; visual mesh filename=package://GC3.1/meshes/link_5.STL
- link link_6: mass 0.349895945126719 -> 0.349895945589167; geometry collision mesh filename=package://GC3.1/meshes/link_6.STL; visual mesh filename=package://GC3.1/meshes/link_6.STL
- link wheel_link_1: geometry collision mesh filename=package://GC3.1/meshes/wheel_link_1.STL; visual mesh filename=package://GC3.1/meshes/wheel_link_1.STL
- link wheel_link_2: geometry collision mesh filename=package://GC3.1/meshes/wheel_link_2.STL; visual mesh filename=package://GC3.1/meshes/wheel_link_2.STL
- link wheel_link_3: geometry collision mesh filename=package://GC3.1/meshes/wheel_link_3.STL; visual mesh filename=package://GC3.1/meshes/wheel_link_3.STL
- link wheel_link_4: geometry collision mesh filename=package://GC3.1/meshes/wheel_link_4.STL; visual mesh filename=package://GC3.1/meshes/wheel_link_4.STL
Joints:
- joint J1: limit lower=-3.14 upper=3.14 effort=0 velocity=0 -> lower=-0.52 upper=1.91 effort=0 velocity=0; origin xyz=0 0 -0.20172 rpy=0 0 0 -> xyz=0 0 -0.106999999999882 rpy=0 0 0
- joint J2: limit lower=-3.14 upper=3.14 effort=0 velocity=0 -> lower=-0.52 upper=2.61 effort=0 velocity=0; origin xyz=0.17397 -0.078842 -0.0545 rpy=-3.1416 0 0 -> xyz=0.1232 0.14596 -0.0545 rpy=3.1416 0 0
- joint J3: origin xyz=-0.070964 0.06903 0 rpy=1.5708 0 0.79921 -> xyz=0.000655997394275049 0.0989978265792674 0 rpy=1.5707963267949 0 -0.00662628479646784
- joint J4: limit lower=-3.14 upper=3.14 effort=0 velocity=0 -> lower=0 upper=1.57 effort=0 velocity=0; origin xyz=-0.00036015 -0.00034683 -0.0465 rpy=-1.5708 -0.97721 -0.80423 -> xyz=-0.000499676236049573 -1.79905288163473E-05 -0.0465000000000025 rpy=-1.5707963267949 0.182122404429995 -1.53480750090966
- joint J5: limit lower=-3.14 upper=3.14 effort=0 velocity=0 -> lower=-1.39 upper=4.36 effort=0 velocity=0; origin xyz=0.022761 0.079818 0 rpy=1.5708 -0.54333 -0.27779 -> xyz=0.0145369266962608 0.0817170591873439 0 rpy=1.57079632679489 -1.53476796314872 -0.176051717388886
- joint J6: limit lower=-3.14 upper=3.14 effort=0 velocity=0 -> lower=-1.57 upper=1.57 effort=0 velocity=0; origin xyz=0.036311 0.023033 -0.0405 rpy=1.5708 0.4276 -1.0055 -> xyz=-0.0429147465036577 -0.00270638735710615 -0.040500000000001 rpy=-1.5707963267949 0.101460063365565 -1.50781545764258
- joint line: limit lower=-1 upper=1 effort=0 velocity=0 -> lower=0 upper=0.38 effort=0 velocity=0; origin xyz=0.0525 0.106 0.216 rpy=3.1416 0 0 -> xyz=0.0524999999999999 0.106 0.216 rpy=3.14159265358979 0 0
- joint wheel_1: origin xyz=0.2935 -0.18 0.08 rpy=-1.5708 0 1.5708 -> xyz=0.2935 -0.18 0.0799999999999999 rpy=-1.5707963267949 0 1.5707963267949
- joint wheel_2: origin xyz=0.2935 0.18 0.08 rpy=-1.5708 0 1.5708 -> xyz=0.2935 0.18 0.0799999999999999 rpy=-1.5707963267949 0 1.5707963267949
- joint wheel_3: origin xyz=-0.2935 -0.18 0.08 rpy=-1.5708 0 1.5708 -> xyz=-0.2935 -0.18 0.0799999999999999 rpy=-1.5707963267949 0 1.5707963267949
- joint wheel_4: origin xyz=-0.2935 0.18 0.08 rpy=-1.5708 0 1.5708 -> xyz=-0.2935 0.18 0.0799999999999999 rpy=-1.5707963267949 0 1.5707963267949

Commit message: 夹爪重新拟合

File: src/runtime/sim/model/rm26_engineer_description/rm26_arm.urdf (robot description, URDF)
Before this commit: robot rm26_arm, 12 links, 11 joints
Links:
- link link_6: mass 0.349895945589167 -> 0.318868553763684

Commit message: 完善26urdf

File: src/runtime/sim/model/rm26_engineer_description/rm26_arm.urdf (robot description, URDF)
Before this commit: robot rm26_arm, 12 links, 11 joints
Links:
- added link arm_base
- added link tcp
Joints:
- added joint arm_base_joint: type fixed, parent line_link, child arm_base, origin xyz=0 0 -0.107 rpy=3.14159265358979 0 0
- added joint tcp_joint: type fixed, parent link_6, child tcp, origin xyz=0.00253 0.08154 0.0438 rpy=3.14159265358979 0 0
